File: Geckonator Dev Edition.kicad_pcb (KiCad board)
At the start: 2 copper layers, 0 parts

Commit message: Added silkscreen, etc.
This corresponds to the first version produced

Signed-off-by: Thomas Flummer <tf@flummer.net>
Parts:
- added C1: CERAMIC-100NF-50V-10%-X7R_0603_, SeeedOPL-Capacitor-2016:C0603, F.Cu at (64.0, 69.4)
- added C2: CERAMIC-100NF-50V-10%-X7R_0603_, SeeedOPL-Capacitor-2016:C0603, F.Cu at (62.0, 69.4)
- added C3: CERAMIC-4.7UF-10V-10%-X5R_0603_, SeeedOPL-Capacitor-2016:C0603, F.Cu at (59.0, 71.0)
- added D1: LED-SMD-RED-DIFFUSED_0603_, SeeedOPL-LED-2016:LED-0603, F.Cu at (73.0, 60.0)
- added D2: SMD-LED-CLEAR-GREEN_0603_, SeeedOPL-LED-2016:LED-0603, F.Cu at (71.0, 60.0)
- added D3: SMD-LED-CLEAR-BLUE_0603_, SeeedOPL-LED-2016:LED-0603, F.Cu at (69.0, 60.0)
- added G***: LOGO, Aesthetics:gecko-14mm, B.Cu at (72.2, 61.3)
- added G***: LOGO, Aesthetics:oshw_logo_5.0mm, B.Cu at (74.0, 74.0)
- added J1: DEBUG, Pin_Headers:Pin_Header_Straight_1x04_Pitch2.54mm, F.Cu at (70.3, 52.4)
- added J2: LE UART, Pin_Headers:Pin_Header_Straight_1x04_Pitch2.54mm, F.Cu at (57.6, 52.4)
- added J3: I2C, Pin_Headers:Pin_Header_Straight_1x04_Pitch2.54mm, F.Cu at (77.9, 57.5)
- added J4: CONN_02X04, Pin_Headers:Pin_Header_Straight_2x04_Pitch2.54mm, F.Cu at (70.3, 88.0)
- added J5: CONN_02X04, Pin_Headers:Pin_Header_Straight_2x04_Pitch2.54mm, F.Cu at (70.3, 95.6)
- added J6: CONN_02X04, Pin_Headers:Pin_Header_Straight_2x04_Pitch2.54mm, F.Cu at (57.6, 95.6)
- added J7: BTNS, Pin_Headers:Pin_Header_Straight_1x04_Pitch2.54mm, F.Cu at (77.9, 70.2)
- added K1: BOOT, SeeedOPL-Switch-2016:SW4-SMD-6.0X6.0X5.0MM, F.Cu at (58.0, 84.0)
- added K2: POWER, SeeedOPL-Switch-2016:SW4-SMD-6.0X6.0X5.0MM, F.Cu at (58.0, 64.0)
- added R1: SMD-RES-1.5K-5%-1_10W_0603_, SeeedOPL-Resistor-2016:R0603, F.Cu at (73.0, 64.0)
- added R2: SMD-RES-1K-5%-1_10W_0603_, SeeedOPL-Resistor-2016:R0603, F.Cu at (71.0, 64.0)
- added R3: SMD-RES-1K-5%-1_10W_0603_, SeeedOPL-Resistor-2016:R0603, F.Cu at (69.0, 64.0)
- added R4: SMD-RES-4.7K-5%-1_10W_0603_, SeeedOPL-Resistor-2016:R0603, F.Cu at (65.8, 83.8)
- added R5: SMD-RES-22R-5%-1_10W_0603_, SeeedOPL-Resistor-2016:R0603, F.Cu at (59.0, 73.0)
- added R6: SMD-RES-22R-5%-1_10W_0603_, SeeedOPL-Resistor-2016:R0603, F.Cu at (59.0, 75.0)
- added REF**: SMD Proto pad, Connectors:SMD_Proto_pad, B.Cu at (95.7, 87.3)
- added REF**: SMD Proto pad, Connectors:SMD_Proto_pad, B.Cu at (95.7, 75.9)
- added REF**: SMD Proto pad, Connectors:SMD_Proto_pad, B.Cu at (98.3, 88.6)
- added REF**: SMD Proto pad, Connectors:SMD_Proto_pad, B.Cu at (98.3, 89.9)
- added REF**: SMD Proto pad, Connectors:SMD_Proto_pad, B.Cu at (98.3, 91.1)
- added REF**: SMD Proto pad, Connectors:SMD_Proto_pad, B.Cu at (95.7, 88.6)
- added REF**: SMD Proto pad, Connectors:SMD_Proto_pad, B.Cu at (95.7, 89.9)
- added REF**: SMD Proto pad, Connectors:SMD_Proto_pad, B.Cu at (95.7, 91.1)
- added REF**: SMD Proto pad, Connectors:SMD_Proto_pad, B.Cu at (93.2, 91.1)
- added REF**: SMD Proto pad, Connectors:SMD_Proto_pad, B.Cu at (93.2, 89.9)
- added REF**: SMD Proto pad, Connectors:SMD_Proto_pad, B.Cu at (93.2, 88.6)
- added REF**: SMD Proto pad, Connectors:SMD_Proto_pad, B.Cu at (93.2, 87.3)
- added REF**: SMD Proto pad, Connectors:SMD_Proto_pad, B.Cu at (95.7, 74.6)
- added REF**: SMD Proto pad, Connectors:SMD_Proto_pad, B.Cu at (93.2, 86.1)
- added REF**: SMD Proto pad, Connectors:SMD_Proto_pad, B.Cu at (93.2, 84.8)
- added REF**: SMD Proto pad, Connectors:SMD_Proto_pad, B.Cu at (93.2, 83.5)
- added REF**: SMD Proto pad, Connectors:SMD_Proto_pad, B.Cu at (93.2, 82.3)
- added REF**: SMD Proto pad, Connectors:SMD_Proto_pad, B.Cu at (93.2, 81.0)
- added REF**: SMD Proto pad, Connectors:SMD_Proto_pad, B.Cu at (93.2, 79.7)
- added REF**: SMD Proto pad, Connectors:SMD_Proto_pad, B.Cu at (93.2, 78.4)
- added REF**: SMD Proto pad, Connectors:SMD_Proto_pad, B.Cu at (93.2, 77.2)
- added REF**: SMD Proto pad, Connectors:SMD_Proto_pad, B.Cu at (93.2, 75.9)
- added REF**: SMD Proto pad, Connectors:SMD_Proto_pad, B.Cu at (93.2, 74.6)
- added REF**: SMD Proto pad, Connectors:SMD_Proto_pad, B.Cu at (95.7, 73.4)
- added REF**: SMD Proto pad, Connectors:SMD_Proto_pad, B.Cu at (93.2, 73.4)
- added REF**: SMD Proto pad, Connectors:SMD_Proto_pad, B.Cu at (93.2, 72.1)
- added REF**: SMD Proto pad, Connectors:SMD_Proto_pad, B.Cu at (93.2, 70.8)
- added REF**: SMD Proto pad, Connectors:SMD_Proto_pad, B.Cu at (93.2, 69.6)
- added REF**: SMD Proto pad, Connectors:SMD_Proto_pad, B.Cu at (93.2, 68.3)
- added REF**: SMD Proto pad, Connectors:SMD_Proto_pad, B.Cu at (93.2, 67.0)
- added REF**: SMD Proto pad, Connectors:SMD_Proto_pad, B.Cu at (93.2, 65.7)
- added REF**: SMD Proto pad, Connectors:SMD_Proto_pad, B.Cu at (90.6, 67.0)
- added REF**: SMD Proto pad, Connectors:SMD_Proto_pad, B.Cu at (90.6, 65.7)
- added REF**: SMD Proto pad, Connectors:SMD_Proto_pad, B.Cu at (90.6, 68.3)
- added REF**: SMD Proto pad, Connectors:SMD_Proto_pad, B.Cu at (95.7, 72.1)
- added REF**: SMD Proto pad, Connectors:SMD_Proto_pad, B.Cu at (90.6, 69.6)
- added REF**: SMD Proto pad, Connectors:SMD_Proto_pad, B.Cu at (90.6, 70.8)
- added REF**: SMD Proto pad, Connectors:SMD_Proto_pad, B.Cu at (90.6, 72.1)
- added REF**: SMD Proto pad, Connectors:SMD_Proto_pad, B.Cu at (90.6, 73.4)
- added REF**: SMD Proto pad, Connectors:SMD_Proto_pad, B.Cu at (90.6, 74.6)
- added REF**: SMD Proto pad, Connectors:SMD_Proto_pad, B.Cu at (90.6, 75.9)
- added REF**: SMD Proto pad, Connectors:SMD_Proto_pad, B.Cu at (90.6, 77.2)
- added REF**: SMD Proto pad, Connectors:SMD_Proto_pad, B.Cu at (90.6, 78.4)
- added REF**: SMD Proto pad, Connectors:SMD_Proto_pad, B.Cu at (90.6, 79.7)
- added REF**: SMD Proto pad, Connectors:SMD_Proto_pad, B.Cu at (90.6, 81.0)
- added REF**: SMD Proto pad, Connectors:SMD_Proto_pad, B.Cu at (95.7, 70.8)
- added REF**: SMD Proto pad, Connectors:SMD_Proto_pad, B.Cu at (90.6, 82.3)
- added REF**: SMD Proto pad, Connectors:SMD_Proto_pad, B.Cu at (90.6, 83.5)
- added REF**: SMD Proto pad, Connectors:SMD_Proto_pad, B.Cu at (90.6, 84.8)
- added REF**: SMD Proto pad, Connectors:SMD_Proto_pad, B.Cu at (90.6, 86.1)
- added REF**: SMD Proto pad, Connectors:SMD_Proto_pad, B.Cu at (90.6, 87.3)
- added REF**: SMD Proto pad, Connectors:SMD_Proto_pad, B.Cu at (90.6, 88.6)
- added REF**: SMD Proto pad, Connectors:SMD_Proto_pad, B.Cu at (90.6, 89.9)
- added REF**: SMD Proto pad, Connectors:SMD_Proto_pad, B.Cu at (90.6, 91.1)
- added REF**: SMD Proto pad, Connectors:SMD_Proto_pad, B.Cu at (88.1, 91.1)
- added REF**: SMD Proto pad, Connectors:SMD_Proto_pad, B.Cu at (88.1, 89.9)
- added REF**: SMD Proto pad, Connectors:SMD_Proto_pad, B.Cu at (95.7, 69.6)
- added REF**: SMD Proto pad, Connectors:SMD_Proto_pad, B.Cu at (88.1, 88.6)
- added REF**: SMD Proto pad, Connectors:SMD_Proto_pad, B.Cu at (88.1, 87.3)
- added REF**: SMD Proto pad, Connectors:SMD_Proto_pad, B.Cu at (88.1, 86.1)
- added REF**: SMD Proto pad, Connectors:SMD_Proto_pad, B.Cu at (88.1, 84.8)
- added REF**: SMD Proto pad, Connectors:SMD_Proto_pad, B.Cu at (88.1, 83.5)
- added REF**: SMD Proto pad, Connectors:SMD_Proto_pad, B.Cu at (88.1, 82.3)
- added REF**: SMD Proto pad, Connectors:SMD_Proto_pad, B.Cu at (88.1, 81.0)
- added REF**: SMD Proto pad, Connectors:SMD_Proto_pad, B.Cu at (88.1, 79.7)
- added REF**: SMD Proto pad, Connectors:SMD_Proto_pad, B.Cu at (88.1, 78.4)
- added REF**: SMD Proto pad, Connectors:SMD_Proto_pad, B.Cu at (88.1, 77.2)
- added REF**: SMD Proto pad, Connectors:SMD_Proto_pad, B.Cu at (95.7, 68.3)
- added REF**: SMD Proto pad, Connectors:SMD_Proto_pad, B.Cu at (88.1, 75.9)
- added REF**: SMD Proto pad, Connectors:SMD_Proto_pad, B.Cu at (88.1, 74.6)
- added REF**: SMD Proto pad, Connectors:SMD_Proto_pad, B.Cu at (88.1, 73.4)
- added REF**: SMD Proto pad, Connectors:SMD_Proto_pad, B.Cu at (88.1, 72.1)
- added REF**: SMD Proto pad, Connectors:SMD_Proto_pad, B.Cu at (88.1, 70.8)
- added REF**: SMD Proto pad, Connectors:SMD_Proto_pad, B.Cu at (88.1, 69.6)
- added REF**: SMD Proto pad, Connectors:SMD_Proto_pad, B.Cu at (88.1, 68.3)
- added REF**: SMD Proto pad, Connectors:SMD_Proto_pad, B.Cu at (88.1, 67.0)
- added REF**: SMD Proto pad, Connectors:SMD_Proto_pad, B.Cu at (88.1, 65.7)
- added REF**: SMD Proto pad, Connectors:SMD_Proto_pad, B.Cu at (85.6, 65.7)
- added REF**: SMD Proto pad, Connectors:SMD_Proto_pad, B.Cu at (95.7, 67.0)
- added REF**: SMD Proto pad, Connectors:SMD_Proto_pad, B.Cu at (85.6, 67.0)
- added REF**: SMD Proto pad, Connectors:SMD_Proto_pad, B.Cu at (85.6, 68.3)
- added REF**: SMD Proto pad, Connectors:SMD_Proto_pad, B.Cu at (85.6, 69.6)
- added REF**: SMD Proto pad, Connectors:SMD_Proto_pad, B.Cu at (85.6, 70.8)
- added REF**: SMD Proto pad, Connectors:SMD_Proto_pad, B.Cu at (85.6, 72.1)
- added REF**: SMD Proto pad, Connectors:SMD_Proto_pad, B.Cu at (85.6, 73.4)
- added REF**: SMD Proto pad, Connectors:SMD_Proto_pad, B.Cu at (85.6, 74.6)
- added REF**: SMD Proto pad, Connectors:SMD_Proto_pad, B.Cu at (85.6, 75.9)
- added REF**: SMD Proto pad, Connectors:SMD_Proto_pad, B.Cu at (85.6, 77.2)
- added REF**: SMD Proto pad, Connectors:SMD_Proto_pad, B.Cu at (85.6, 78.4)
- added REF**: SMD Proto pad, Connectors:SMD_Proto_pad, B.Cu at (95.7, 65.7)
- added REF**: SMD Proto pad, Connectors:SMD_Proto_pad, B.Cu at (85.6, 79.7)
- added REF**: SMD Proto pad, Connectors:SMD_Proto_pad, B.Cu at (85.6, 81.0)
- added REF**: SMD Proto pad, Connectors:SMD_Proto_pad, B.Cu at (85.6, 82.3)
- added REF**: SMD Proto pad, Connectors:SMD_Proto_pad, B.Cu at (85.6, 83.5)
- added REF**: SMD Proto pad, Connectors:SMD_Proto_pad, B.Cu at (85.6, 84.8)
- added REF**: SMD Proto pad, Connectors:SMD_Proto_pad, B.Cu at (85.6, 86.1)
- added REF**: SMD Proto pad, Connectors:SMD_Proto_pad, B.Cu at (85.6, 87.3)
- added REF**: SMD Proto pad, Connectors:SMD_Proto_pad, B.Cu at (85.6, 88.6)
- added REF**: SMD Proto pad, Connectors:SMD_Proto_pad, B.Cu at (85.6, 89.9)
- added REF**: SMD Proto pad, Connectors:SMD_Proto_pad, B.Cu at (85.6, 91.1)
- added REF**: SMD Proto pad, Connectors:SMD_Proto_pad, B.Cu at (98.3, 65.7)
- added REF**: SMD Proto pad, Connectors:SMD_Proto_pad, B.Cu at (83.0, 91.1)
- added REF**: SMD Proto pad, Connectors:SMD_Proto_pad, B.Cu at (83.0, 89.9)
- added REF**: SMD Proto pad, Connectors:SMD_Proto_pad, B.Cu at (83.0, 88.6)
- added REF**: SMD Proto pad, Connectors:SMD_Proto_pad, B.Cu at (83.0, 87.3)
- added REF**: SMD Proto pad, Connectors:SMD_Proto_pad, B.Cu at (83.0, 86.1)
- added REF**: SMD Proto pad, Connectors:SMD_Proto_pad, B.Cu at (83.0, 84.8)
- added REF**: SMD Proto pad, Connectors:SMD_Proto_pad, B.Cu at (83.0, 83.5)
- added REF**: SMD Proto pad, Connectors:SMD_Proto_pad, B.Cu at (83.0, 82.3)
- added REF**: SMD Proto pad, Connectors:SMD_Proto_pad, B.Cu at (83.0, 81.0)
- added REF**: SMD Proto pad, Connectors:SMD_Proto_pad, B.Cu at (83.0, 79.7)
- added REF**: SMD Proto pad, Connectors:SMD_Proto_pad, B.Cu at (95.7, 86.1)
- added REF**: SMD Proto pad, Connectors:SMD_Proto_pad, B.Cu at (98.3, 67.0)
- added REF**: SMD Proto pad, Connectors:SMD_Proto_pad, B.Cu at (83.0, 78.4)
- added REF**: SMD Proto pad, Connectors:SMD_Proto_pad, B.Cu at (83.0, 77.2)
- added REF**: SMD Proto pad, Connectors:SMD_Proto_pad, B.Cu at (83.0, 75.9)
- added REF**: SMD Proto pad, Connectors:SMD_Proto_pad, B.Cu at (83.0, 74.6)
- added REF**: SMD Proto pad, Connectors:SMD_Proto_pad, B.Cu at (83.0, 73.4)
- added REF**: SMD Proto pad, Connectors:SMD_Proto_pad, B.Cu at (83.0, 72.1)
- added REF**: SMD Proto pad, Connectors:SMD_Proto_pad, B.Cu at (83.0, 70.8)
- added REF**: SMD Proto pad, Connectors:SMD_Proto_pad, B.Cu at (83.0, 69.6)
- added REF**: SMD Proto pad, Connectors:SMD_Proto_pad, B.Cu at (83.0, 68.3)
- added REF**: SMD Proto pad, Connectors:SMD_Proto_pad, B.Cu at (83.0, 67.0)
- added REF**: SMD Proto pad, Connectors:SMD_Proto_pad, B.Cu at (98.3, 68.3)
- added REF**: SMD Proto pad, Connectors:SMD_Proto_pad, B.Cu at (105.9, 64.5)
- added REF**: SMD Proto pad, Connectors:SMD_Proto_pad, B.Cu at (103.3, 64.5)
- added REF**: SMD Proto pad, Connectors:SMD_Proto_pad, B.Cu at (100.8, 64.5)
- added REF**: SMD Proto pad, Connectors:SMD_Proto_pad, B.Cu at (98.3, 64.5)
- added REF**: SMD Proto pad, Connectors:SMD_Proto_pad, B.Cu at (95.7, 64.5)
- added REF**: SMD Proto pad, Connectors:SMD_Proto_pad, B.Cu at (93.2, 64.5)
- added REF**: SMD Proto pad, Connectors:SMD_Proto_pad, B.Cu at (90.6, 64.5)
- added REF**: SMD Proto pad, Connectors:SMD_Proto_pad, B.Cu at (88.1, 64.5)
- added REF**: SMD Proto pad, Connectors:SMD_Proto_pad, B.Cu at (85.6, 64.5)
- added REF**: SMD Proto pad, Connectors:SMD_Proto_pad, B.Cu at (83.0, 65.7)
- added REF**: SMD Proto pad, Connectors:SMD_Proto_pad, B.Cu at (98.3, 69.6)
- added REF**: SMD Proto pad, Connectors:SMD_Proto_pad, B.Cu at (83.0, 64.5)
- added REF**: SMD Proto pad, Connectors:SMD_Proto_pad, B.Cu at (83.0, 63.2)
- added REF**: SMD Proto pad, Connectors:SMD_Proto_pad, B.Cu at (85.6, 63.2)
- added REF**: SMD Proto pad, Connectors:SMD_Proto_pad, B.Cu at (88.1, 63.2)
- added REF**: SMD Proto pad, Connectors:SMD_Proto_pad, B.Cu at (90.6, 63.2)
- added REF**: SMD Proto pad, Connectors:SMD_Proto_pad, B.Cu at (93.2, 63.2)
- added REF**: SMD Proto pad, Connectors:SMD_Proto_pad, B.Cu at (95.7, 63.2)
- added REF**: SMD Proto pad, Connectors:SMD_Proto_pad, B.Cu at (98.3, 63.2)
- added REF**: SMD Proto pad, Connectors:SMD_Proto_pad, B.Cu at (100.8, 63.2)
- added REF**: SMD Proto pad, Connectors:SMD_Proto_pad, B.Cu at (103.3, 63.2)
- added REF**: SMD Proto pad, Connectors:SMD_Proto_pad, B.Cu at (98.3, 70.8)
- added REF**: SMD Proto pad, Connectors:SMD_Proto_pad, B.Cu at (105.9, 63.2)
- added REF**: SMD Proto pad, Connectors:SMD_Proto_pad, B.Cu at (105.9, 61.9)
- added REF**: SMD Proto pad, Connectors:SMD_Proto_pad, B.Cu at (103.3, 61.9)
- added REF**: SMD Proto pad, Connectors:SMD_Proto_pad, B.Cu at (100.8, 61.9)
- added REF**: SMD Proto pad, Connectors:SMD_Proto_pad, B.Cu at (98.3, 61.9)
- added REF**: SMD Proto pad, Connectors:SMD_Proto_pad, B.Cu at (95.7, 61.9)
- added REF**: SMD Proto pad, Connectors:SMD_Proto_pad, B.Cu at (93.2, 61.9)
- added REF**: SMD Proto pad, Connectors:SMD_Proto_pad, B.Cu at (90.6, 61.9)
- added REF**: SMD Proto pad, Connectors:SMD_Proto_pad, B.Cu at (88.1, 61.9)
- added REF**: SMD Proto pad, Connectors:SMD_Proto_pad, B.Cu at (85.6, 61.9)
- added REF**: SMD Proto pad, Connectors:SMD_Proto_pad, B.Cu at (98.3, 72.1)
- added REF**: SMD Proto pad, Connectors:SMD_Proto_pad, B.Cu at (83.0, 61.9)
- added REF**: SMD Proto pad, Connectors:SMD_Proto_pad, B.Cu at (83.0, 60.7)
- added REF**: SMD Proto pad, Connectors:SMD_Proto_pad, B.Cu at (85.6, 60.7)
- added REF**: SMD Proto pad, Connectors:SMD_Proto_pad, B.Cu at (88.1, 60.7)
- added REF**: SMD Proto pad, Connectors:SMD_Proto_pad, B.Cu at (90.6, 60.7)
- added REF**: SMD Proto pad, Connectors:SMD_Proto_pad, B.Cu at (93.2, 60.7)
- added REF**: SMD Proto pad, Connectors:SMD_Proto_pad, B.Cu at (95.7, 60.7)
- added REF**: SMD Proto pad, Connectors:SMD_Proto_pad, B.Cu at (98.3, 60.7)
- added REF**: SMD Proto pad, Connectors:SMD_Proto_pad, B.Cu at (100.8, 60.7)
- added REF**: SMD Proto pad, Connectors:SMD_Proto_pad, B.Cu at (103.3, 60.7)
- added REF**: SMD Proto pad, Connectors:SMD_Proto_pad, B.Cu at (98.3, 73.4)
- added REF**: SMD Proto pad, Connectors:SMD_Proto_pad, B.Cu at (105.9, 60.7)
- added REF**: SMD Proto pad, Connectors:SMD_Proto_pad, B.Cu at (105.9, 59.4)
- added REF**: SMD Proto pad, Connectors:SMD_Proto_pad, B.Cu at (103.3, 59.4)
- added REF**: SMD Proto pad, Connectors:SMD_Proto_pad, B.Cu at (100.8, 59.4)
- added REF**: SMD Proto pad, Connectors:SMD_Proto_pad, B.Cu at (98.3, 59.4)
- added REF**: SMD Proto pad, Connectors:SMD_Proto_pad, B.Cu at (95.7, 59.4)
- added REF**: SMD Proto pad, Connectors:SMD_Proto_pad, B.Cu at (93.2, 59.4)
- added REF**: SMD Proto pad, Connectors:SMD_Proto_pad, B.Cu at (90.6, 59.4)
- added REF**: SMD Proto pad, Connectors:SMD_Proto_pad, B.Cu at (88.1, 59.4)
- added REF**: SMD Proto pad, Connectors:SMD_Proto_pad, B.Cu at (85.6, 59.4)
- added REF**: SMD Proto pad, Connectors:SMD_Proto_pad, B.Cu at (98.3, 74.6)
- added REF**: SMD Proto pad, Connectors:SMD_Proto_pad, B.Cu at (83.0, 59.4)
- added REF**: SMD Proto pad, Connectors:SMD_Proto_pad, B.Cu at (83.0, 58.1)
- added REF**: SMD Proto pad, Connectors:SMD_Proto_pad, B.Cu at (85.6, 58.1)
- added REF**: SMD Proto pad, Connectors:SMD_Proto_pad, B.Cu at (88.1, 58.1)
- added REF**: SMD Proto pad, Connectors:SMD_Proto_pad, B.Cu at (90.6, 58.1)
- added REF**: SMD Proto pad, Connectors:SMD_Proto_pad, B.Cu at (93.2, 58.1)
- added REF**: SMD Proto pad, Connectors:SMD_Proto_pad, B.Cu at (95.7, 58.1)
- added REF**: SMD Proto pad, Connectors:SMD_Proto_pad, B.Cu at (98.3, 58.1)
- added REF**: SMD Proto pad, Connectors:SMD_Proto_pad, B.Cu at (100.8, 58.1)
- added REF**: SMD Proto pad, Connectors:SMD_Proto_pad, B.Cu at (103.3, 58.1)
- added REF**: SMD Proto pad, Connectors:SMD_Proto_pad, B.Cu at (98.3, 75.9)
- added REF**: SMD Proto pad, Connectors:SMD_Proto_pad, B.Cu at (105.9, 58.1)
- added REF**: SMD Proto pad, Connectors:SMD_Proto_pad, B.Cu at (105.9, 56.9)
- added REF**: SMD Proto pad, Connectors:SMD_Proto_pad, B.Cu at (103.3, 56.9)
- added REF**: SMD Proto pad, Connectors:SMD_Proto_pad, B.Cu at (100.8, 56.9)
- added REF**: SMD Proto pad, Connectors:SMD_Proto_pad, B.Cu at (98.3, 56.9)
- added REF**: SMD Proto pad, Connectors:SMD_Proto_pad, B.Cu at (95.7, 56.9)
- added REF**: SMD Proto pad, Connectors:SMD_Proto_pad, B.Cu at (93.2, 56.9)
- added REF**: SMD Proto pad, Connectors:SMD_Proto_pad, B.Cu at (90.6, 56.9)
- added REF**: SMD Proto pad, Connectors:SMD_Proto_pad, B.Cu at (88.1, 56.9)
- added REF**: SMD Proto pad, Connectors:SMD_Proto_pad, B.Cu at (85.6, 56.9)
- added REF**: SMD Proto pad, Connectors:SMD_Proto_pad, B.Cu at (98.3, 77.2)
- added REF**: SMD Proto pad, Connectors:SMD_Proto_pad, F.Cu at (106.5, 90.5)
- added REF**: SMD Proto pad, Connectors:SMD_Proto_pad, F.Cu at (105.2, 90.5)
- added REF**: SMD Proto pad, Connectors:SMD_Proto_pad, F.Cu at (104.0, 90.5)
- added REF**: SMD Proto pad, Connectors:SMD_Proto_pad, F.Cu at (102.7, 90.5)
- added REF**: SMD Proto pad, Connectors:SMD_Proto_pad, F.Cu at (101.4, 90.5)
- added REF**: SMD Proto pad, Connectors:SMD_Proto_pad, F.Cu at (100.2, 90.5)
- added REF**: SMD Proto pad, Connectors:SMD_Proto_pad, F.Cu at (98.9, 90.5)
- added REF**: SMD Proto pad, Connectors:SMD_Proto_pad, F.Cu at (97.6, 90.5)
- added REF**: SMD Proto pad, Connectors:SMD_Proto_pad, F.Cu at (96.4, 90.5)
- added REF**: SMD Proto pad, Connectors:SMD_Proto_pad, F.Cu at (95.1, 90.5)
- added REF**: SMD Proto pad, Connectors:SMD_Proto_pad, B.Cu at (98.3, 78.4)
- added REF**: SMD Proto pad, Connectors:SMD_Proto_pad, F.Cu at (93.8, 90.5)
- added REF**: SMD Proto pad, Connectors:SMD_Proto_pad, F.Cu at (92.5, 90.5)
- added REF**: SMD Proto pad, Connectors:SMD_Proto_pad, F.Cu at (91.3, 90.5)
- added REF**: SMD Proto pad, Connectors:SMD_Proto_pad, F.Cu at (90.0, 90.5)
- added REF**: SMD Proto pad, Connectors:SMD_Proto_pad, F.Cu at (88.7, 90.5)
- added REF**: SMD Proto pad, Connectors:SMD_Proto_pad, F.Cu at (87.5, 90.5)
- added REF**: SMD Proto pad, Connectors:SMD_Proto_pad, F.Cu at (86.2, 90.5)
- added REF**: SMD Proto pad, Connectors:SMD_Proto_pad, F.Cu at (84.9, 90.5)
- added REF**: SMD Proto pad, Connectors:SMD_Proto_pad, F.Cu at (83.7, 90.5)
- added REF**: SMD Proto pad, Connectors:SMD_Proto_pad, F.Cu at (82.4, 90.5)
- added REF**: SMD Proto pad, Connectors:SMD_Proto_pad, B.Cu at (95.7, 84.8)
- added REF**: SMD Proto pad, Connectors:SMD_Proto_pad, B.Cu at (98.3, 79.7)
- added REF**: SMD Proto pad, Connectors:SMD_Proto_pad, F.Cu at (106.5, 57.5)
- added REF**: SMD Proto pad, Connectors:SMD_Proto_pad, F.Cu at (105.2, 57.5)
- added REF**: SMD Proto pad, Connectors:SMD_Proto_pad, F.Cu at (104.0, 57.5)
- added REF**: SMD Proto pad, Connectors:SMD_Proto_pad, F.Cu at (102.7, 57.5)
- added REF**: SMD Proto pad, Connectors:SMD_Proto_pad, F.Cu at (101.4, 57.5)
- added REF**: SMD Proto pad, Connectors:SMD_Proto_pad, F.Cu at (100.2, 57.5)
- added REF**: SMD Proto pad, Connectors:SMD_Proto_pad, F.Cu at (98.9, 57.5)
- added REF**: SMD Proto pad, Connectors:SMD_Proto_pad, F.Cu at (97.6, 57.5)
- added REF**: SMD Proto pad, Connectors:SMD_Proto_pad, F.Cu at (96.4, 57.5)
- added REF**: SMD Proto pad, Connectors:SMD_Proto_pad, F.Cu at (95.1, 57.5)
- added REF**: SMD Proto pad, Connectors:SMD_Proto_pad, B.Cu at (98.3, 81.0)
- added REF**: SMD Proto pad, Connectors:SMD_Proto_pad, F.Cu at (93.8, 57.5)
- added REF**: SMD Proto pad, Connectors:SMD_Proto_pad, F.Cu at (92.5, 57.5)
- added REF**: SMD Proto pad, Connectors:SMD_Proto_pad, F.Cu at (91.3, 57.5)
- added REF**: SMD Proto pad, Connectors:SMD_Proto_pad, F.Cu at (90.0, 57.5)
- added REF**: SMD Proto pad, Connectors:SMD_Proto_pad, F.Cu at (88.7, 57.5)
- added REF**: SMD Proto pad, Connectors:SMD_Proto_pad, F.Cu at (87.5, 57.5)
- added REF**: SMD Proto pad, Connectors:SMD_Proto_pad, F.Cu at (86.2, 57.5)
- added REF**: SMD Proto pad, Connectors:SMD_Proto_pad, F.Cu at (84.9, 57.5)
- added REF**: SMD Proto pad, Connectors:SMD_Proto_pad, F.Cu at (83.7, 57.5)
- added REF**: SMD Proto pad, Connectors:SMD_Proto_pad, F.Cu at (82.4, 57.5)
- added REF**: SMD Proto pad, Connectors:SMD_Proto_pad, B.Cu at (98.3, 82.3)
- added REF**: SMD Proto pad, Connectors:SMD_Proto_pad, F.Cu at (106.5, 72.7)
- added REF**: SMD Proto pad, Connectors:SMD_Proto_pad, F.Cu at (105.2, 72.7)
- added REF**: SMD Proto pad, Connectors:SMD_Proto_pad, F.Cu at (104.0, 72.7)
- added REF**: SMD Proto pad, Connectors:SMD_Proto_pad, F.Cu at (102.7, 72.7)
- added REF**: SMD Proto pad, Connectors:SMD_Proto_pad, F.Cu at (101.4, 72.7)
- added REF**: SMD Proto pad, Connectors:SMD_Proto_pad, F.Cu at (100.2, 72.7)
- added REF**: SMD Proto pad, Connectors:SMD_Proto_pad, F.Cu at (98.9, 72.7)
- added REF**: SMD Proto pad, Connectors:SMD_Proto_pad, F.Cu at (97.6, 72.7)
- added REF**: SMD Proto pad, Connectors:SMD_Proto_pad, F.Cu at (96.4, 72.7)
- added REF**: SMD Proto pad, Connectors:SMD_Proto_pad, F.Cu at (95.1, 72.7)
- added REF**: SMD Proto pad, Connectors:SMD_Proto_pad, B.Cu at (98.3, 83.5)
- added REF**: SMD Proto pad, Connectors:SMD_Proto_pad, F.Cu at (93.8, 72.7)
- added REF**: SMD Proto pad, Connectors:SMD_Proto_pad, F.Cu at (92.5, 72.7)
- added REF**: SMD Proto pad, Connectors:SMD_Proto_pad, F.Cu at (91.3, 72.7)
- added REF**: SMD Proto pad, Connectors:SMD_Proto_pad, F.Cu at (90.0, 72.7)
- added REF**: SMD Proto pad, Connectors:SMD_Proto_pad, F.Cu at (88.7, 72.7)
- added REF**: SMD Proto pad, Connectors:SMD_Proto_pad, F.Cu at (87.5, 72.7)
- added REF**: SMD Proto pad, Connectors:SMD_Proto_pad, F.Cu at (86.2, 72.7)
- added REF**: SMD Proto pad, Connectors:SMD_Proto_pad, F.Cu at (84.9, 72.7)
- added REF**: SMD Proto pad, Connectors:SMD_Proto_pad, F.Cu at (83.7, 72.7)
- added REF**: SMD Proto pad, Connectors:SMD_Proto_pad, F.Cu at (82.4, 72.7)
- added REF**: SMD Proto pad, Connectors:SMD_Proto_pad, B.Cu at (98.3, 84.8)
- added REF**: SMD Proto pad, Connectors:SMD_Proto_pad, F.Cu at (106.5, 75.3)
- added REF**: SMD Proto pad, Connectors:SMD_Proto_pad, F.Cu at (105.2, 75.3)
- added REF**: SMD Proto pad, Connectors:SMD_Proto_pad, F.Cu at (104.0, 75.3)
- added REF**: SMD Proto pad, Connectors:SMD_Proto_pad, F.Cu at (102.7, 75.3)
- added REF**: SMD Proto pad, Connectors:SMD_Proto_pad, F.Cu at (101.4, 75.3)
- added REF**: SMD Proto pad, Connectors:SMD_Proto_pad, F.Cu at (100.2, 75.3)
- added REF**: SMD Proto pad, Connectors:SMD_Proto_pad, F.Cu at (98.9, 75.3)
- added REF**: SMD Proto pad, Connectors:SMD_Proto_pad, F.Cu at (97.6, 75.3)
- added REF**: SMD Proto pad, Connectors:SMD_Proto_pad, F.Cu at (96.4, 75.3)
- added REF**: SMD Proto pad, Connectors:SMD_Proto_pad, F.Cu at (95.1, 75.3)
- added REF**: SMD Proto pad, Connectors:SMD_Proto_pad, B.Cu at (98.3, 86.1)
- added REF**: SMD Proto pad, Connectors:SMD_Proto_pad, F.Cu at (93.8, 75.3)
- added REF**: SMD Proto pad, Connectors:SMD_Proto_pad, F.Cu at (92.5, 75.3)
- added REF**: SMD Proto pad, Connectors:SMD_Proto_pad, F.Cu at (91.3, 75.3)
- added REF**: SMD Proto pad, Connectors:SMD_Proto_pad, F.Cu at (90.0, 75.3)
- added REF**: SMD Proto pad, Connectors:SMD_Proto_pad, F.Cu at (88.7, 75.3)
- added REF**: SMD Proto pad, Connectors:SMD_Proto_pad, F.Cu at (87.5, 75.3)
- added REF**: SMD Proto pad, Connectors:SMD_Proto_pad, F.Cu at (86.2, 75.3)
- added REF**: SMD Proto pad, Connectors:SMD_Proto_pad, F.Cu at (84.9, 75.3)
- added REF**: SMD Proto pad, Connectors:SMD_Proto_pad, F.Cu at (83.7, 75.3)
- added REF**: SMD Proto pad, Connectors:SMD_Proto_pad, F.Cu at (82.4, 75.3)
- added REF**: SMD Proto pad, Connectors:SMD_Proto_pad, B.Cu at (98.3, 87.3)
- added REF**: SMD Proto pad, Connectors:SMD_Proto_pad, F.Cu at (106.5, 77.8)
- added REF**: SMD Proto pad, Connectors:SMD_Proto_pad, F.Cu at (105.2, 77.8)
- added REF**: SMD Proto pad, Connectors:SMD_Proto_pad, F.Cu at (104.0, 77.8)
- added REF**: SMD Proto pad, Connectors:SMD_Proto_pad, F.Cu at (102.7, 77.8)
- added REF**: SMD Proto pad, Connectors:SMD_Proto_pad, F.Cu at (101.4, 77.8)
- added REF**: SMD Proto pad, Connectors:SMD_Proto_pad, F.Cu at (100.2, 77.8)
- added REF**: SMD Proto pad, Connectors:SMD_Proto_pad, F.Cu at (98.9, 77.8)
- added REF**: SMD Proto pad, Connectors:SMD_Proto_pad, F.Cu at (97.6, 77.8)
- added REF**: SMD Proto pad, Connectors:SMD_Proto_pad, F.Cu at (96.4, 77.8)
- added REF**: SMD Proto pad, Connectors:SMD_Proto_pad, F.Cu at (95.1, 77.8)
- added REF**: SMD Proto pad, Connectors:SMD_Proto_pad, B.Cu at (100.8, 87.3)
- added REF**: SMD Proto pad, Connectors:SMD_Proto_pad, F.Cu at (93.8, 77.8)
- added REF**: SMD Proto pad, Connectors:SMD_Proto_pad, F.Cu at (92.5, 77.8)
- added REF**: SMD Proto pad, Connectors:SMD_Proto_pad, F.Cu at (91.3, 77.8)
- added REF**: SMD Proto pad, Connectors:SMD_Proto_pad, F.Cu at (90.0, 77.8)
- added REF**: SMD Proto pad, Connectors:SMD_Proto_pad, F.Cu at (88.7, 77.8)
- added REF**: SMD Proto pad, Connectors:SMD_Proto_pad, F.Cu at (87.5, 77.8)
- added REF**: SMD Proto pad, Connectors:SMD_Proto_pad, F.Cu at (86.2, 77.8)
- added REF**: SMD Proto pad, Connectors:SMD_Proto_pad, F.Cu at (84.9, 77.8)
- added REF**: SMD Proto pad, Connectors:SMD_Proto_pad, F.Cu at (83.7, 77.8)
- added REF**: SMD Proto pad, Connectors:SMD_Proto_pad, F.Cu at (82.4, 77.8)
- added REF**: SMD Proto pad, Connectors:SMD_Proto_pad, B.Cu at (100.8, 86.1)
- added REF**: SMD Proto pad, Connectors:SMD_Proto_pad, F.Cu at (106.5, 80.3)
- added REF**: SMD Proto pad, Connectors:SMD_Proto_pad, F.Cu at (105.2, 80.3)
- added REF**: SMD Proto pad, Connectors:SMD_Proto_pad, F.Cu at (104.0, 80.3)
- added REF**: SMD Proto pad, Connectors:SMD_Proto_pad, F.Cu at (102.7, 80.3)
- added REF**: SMD Proto pad, Connectors:SMD_Proto_pad, F.Cu at (101.4, 80.3)
- added REF**: SMD Proto pad, Connectors:SMD_Proto_pad, F.Cu at (100.2, 80.3)
- added REF**: SMD Proto pad, Connectors:SMD_Proto_pad, F.Cu at (98.9, 80.3)
- added REF**: SMD Proto pad, Connectors:SMD_Proto_pad, F.Cu at (97.6, 80.3)
- added REF**: SMD Proto pad, Connectors:SMD_Proto_pad, F.Cu at (96.4, 80.3)
- added REF**: SMD Proto pad, Connectors:SMD_Proto_pad, F.Cu at (95.1, 80.3)
- added REF**: SMD Proto pad, Connectors:SMD_Proto_pad, B.Cu at (100.8, 84.8)
- added REF**: SMD Proto pad, Connectors:SMD_Proto_pad, F.Cu at (93.8, 80.3)
- added REF**: SMD Proto pad, Connectors:SMD_Proto_pad, F.Cu at (92.5, 80.3)
- added REF**: SMD Proto pad, Connectors:SMD_Proto_pad, F.Cu at (91.3, 80.3)
- added REF**: SMD Proto pad, Connectors:SMD_Proto_pad, F.Cu at (90.0, 80.3)
- added REF**: SMD Proto pad, Connectors:SMD_Proto_pad, F.Cu at (88.7, 80.3)
- added REF**: SMD Proto pad, Connectors:SMD_Proto_pad, F.Cu at (87.5, 80.3)
- added REF**: SMD Proto pad, Connectors:SMD_Proto_pad, F.Cu at (86.2, 80.3)
- added REF**: SMD Proto pad, Connectors:SMD_Proto_pad, F.Cu at (84.9, 80.3)
- added REF**: SMD Proto pad, Connectors:SMD_Proto_pad, F.Cu at (83.7, 80.3)
- added REF**: SMD Proto pad, Connectors:SMD_Proto_pad, F.Cu at (82.4, 80.3)
- added REF**: SMD Proto pad, Connectors:SMD_Proto_pad, B.Cu at (95.7, 83.5)
- added REF**: SMD Proto pad, Connectors:SMD_Proto_pad, B.Cu at (100.8, 83.5)
- added REF**: SMD Proto pad, Connectors:SMD_Proto_pad, F.Cu at (106.5, 82.9)
- added REF**: SMD Proto pad, Connectors:SMD_Proto_pad, F.Cu at (105.2, 82.9)
- added REF**: SMD Proto pad, Connectors:SMD_Proto_pad, F.Cu at (104.0, 82.9)
- added REF**: SMD Proto pad, Connectors:SMD_Proto_pad, F.Cu at (102.7, 82.9)
- added REF**: SMD Proto pad, Connectors:SMD_Proto_pad, F.Cu at (101.4, 82.9)
- added REF**: SMD Proto pad, Connectors:SMD_Proto_pad, F.Cu at (100.2, 82.9)
- added REF**: SMD Proto pad, Connectors:SMD_Proto_pad, F.Cu at (98.9, 82.9)
- added REF**: SMD Proto pad, Connectors:SMD_Proto_pad, F.Cu at (97.6, 82.9)
- added REF**: SMD Proto pad, Connectors:SMD_Proto_pad, F.Cu at (96.4, 82.9)
- added REF**: SMD Proto pad, Connectors:SMD_Proto_pad, F.Cu at (95.1, 82.9)
- added REF**: SMD Proto pad, Connectors:SMD_Proto_pad, B.Cu at (100.8, 82.3)
- added REF**: SMD Proto pad, Connectors:SMD_Proto_pad, F.Cu at (93.8, 82.9)
- added REF**: SMD Proto pad, Connectors:SMD_Proto_pad, F.Cu at (92.5, 82.9)
- added REF**: SMD Proto pad, Connectors:SMD_Proto_pad, F.Cu at (91.3, 82.9)
- added REF**: SMD Proto pad, Connectors:SMD_Proto_pad, F.Cu at (90.0, 82.9)
- added REF**: SMD Proto pad, Connectors:SMD_Proto_pad, F.Cu at (88.7, 82.9)
- added REF**: SMD Proto pad, Connectors:SMD_Proto_pad, F.Cu at (87.5, 82.9)
- added REF**: SMD Proto pad, Connectors:SMD_Proto_pad, F.Cu at (86.2, 82.9)
- added REF**: SMD Proto pad, Connectors:SMD_Proto_pad, F.Cu at (84.9, 82.9)
- added REF**: SMD Proto pad, Connectors:SMD_Proto_pad, F.Cu at (83.7, 82.9)
- added REF**: SMD Proto pad, Connectors:SMD_Proto_pad, F.Cu at (82.4, 82.9)
- added REF**: SMD Proto pad, Connectors:SMD_Proto_pad, B.Cu at (100.8, 81.0)
- added REF**: SMD Proto pad, Connectors:SMD_Proto_pad, F.Cu at (106.5, 85.4)
- added REF**: SMD Proto pad, Connectors:SMD_Proto_pad, F.Cu at (105.2, 85.4)
- added REF**: SMD Proto pad, Connectors:SMD_Proto_pad, F.Cu at (104.0, 85.4)
- added REF**: SMD Proto pad, Connectors:SMD_Proto_pad, F.Cu at (102.7, 85.4)
- added REF**: SMD Proto pad, Connectors:SMD_Proto_pad, F.Cu at (101.4, 85.4)
- added REF**: SMD Proto pad, Connectors:SMD_Proto_pad, F.Cu at (100.2, 85.4)
- added REF**: SMD Proto pad, Connectors:SMD_Proto_pad, F.Cu at (98.9, 85.4)
- added REF**: SMD Proto pad, Connectors:SMD_Proto_pad, F.Cu at (97.6, 85.4)
- added REF**: SMD Proto pad, Connectors:SMD_Proto_pad, F.Cu at (96.4, 85.4)
- added REF**: SMD Proto pad, Connectors:SMD_Proto_pad, F.Cu at (95.1, 85.4)
- added REF**: SMD Proto pad, Connectors:SMD_Proto_pad, B.Cu at (100.8, 79.7)
- added REF**: SMD Proto pad, Connectors:SMD_Proto_pad, F.Cu at (93.8, 85.4)
- added REF**: SMD Proto pad, Connectors:SMD_Proto_pad, F.Cu at (92.5, 85.4)
- added REF**: SMD Proto pad, Connectors:SMD_Proto_pad, F.Cu at (91.3, 85.4)
- added REF**: SMD Proto pad, Connectors:SMD_Proto_pad, F.Cu at (90.0, 85.4)
- added REF**: SMD Proto pad, Connectors:SMD_Proto_pad, F.Cu at (88.7, 85.4)
- added REF**: SMD Proto pad, Connectors:SMD_Proto_pad, F.Cu at (87.5, 85.4)
- added REF**: SMD Proto pad, Connectors:SMD_Proto_pad, F.Cu at (86.2, 85.4)
- added REF**: SMD Proto pad, Connectors:SMD_Proto_pad, F.Cu at (84.9, 85.4)
- added REF**: SMD Proto pad, Connectors:SMD_Proto_pad, F.Cu at (83.7, 85.4)
- added REF**: SMD Proto pad, Connectors:SMD_Proto_pad, F.Cu at (82.4, 85.4)
- added REF**: SMD Proto pad, Connectors:SMD_Proto_pad, B.Cu at (100.8, 78.4)
- added REF**: SMD Proto pad, Connectors:SMD_Proto_pad, F.Cu at (106.5, 88.0)
- added REF**: SMD Proto pad, Connectors:SMD_Proto_pad, F.Cu at (105.2, 88.0)
- added REF**: SMD Proto pad, Connectors:SMD_Proto_pad, F.Cu at (104.0, 88.0)
- added REF**: SMD Proto pad, Connectors:SMD_Proto_pad, F.Cu at (102.7, 88.0)
- added REF**: SMD Proto pad, Connectors:SMD_Proto_pad, F.Cu at (101.4, 88.0)
- added REF**: SMD Proto pad, Connectors:SMD_Proto_pad, F.Cu at (100.2, 88.0)
- added REF**: SMD Proto pad, Connectors:SMD_Proto_pad, F.Cu at (98.9, 88.0)
- added REF**: SMD Proto pad, Connectors:SMD_Proto_pad, F.Cu at (97.6, 88.0)
- added REF**: SMD Proto pad, Connectors:SMD_Proto_pad, F.Cu at (96.4, 88.0)
- added REF**: SMD Proto pad, Connectors:SMD_Proto_pad, F.Cu at (95.1, 88.0)
- added REF**: SMD Proto pad, Connectors:SMD_Proto_pad, B.Cu at (100.8, 77.2)
- added REF**: SMD Proto pad, Connectors:SMD_Proto_pad, F.Cu at (93.8, 88.0)
- added REF**: SMD Proto pad, Connectors:SMD_Proto_pad, F.Cu at (92.5, 88.0)
- added REF**: SMD Proto pad, Connectors:SMD_Proto_pad, F.Cu at (91.3, 88.0)
- added REF**: SMD Proto pad, Connectors:SMD_Proto_pad, F.Cu at (90.0, 88.0)
- added REF**: SMD Proto pad, Connectors:SMD_Proto_pad, F.Cu at (88.7, 88.0)
- added REF**: SMD Proto pad, Connectors:SMD_Proto_pad, F.Cu at (87.5, 88.0)
- added REF**: SMD Proto pad, Connectors:SMD_Proto_pad, F.Cu at (86.2, 88.0)
- added REF**: SMD Proto pad, Connectors:SMD_Proto_pad, F.Cu at (84.9, 88.0)
- added REF**: SMD Proto pad, Connectors:SMD_Proto_pad, F.Cu at (83.7, 88.0)
- added REF**: SMD Proto pad, Connectors:SMD_Proto_pad, F.Cu at (82.4, 88.0)
- added REF**: SMD Proto pad, Connectors:SMD_Proto_pad, B.Cu at (100.8, 75.9)
- added REF**: SMD Proto pad, Connectors:SMD_Proto_pad, F.Cu at (106.5, 70.2)
- added REF**: SMD Proto pad, Connectors:SMD_Proto_pad, F.Cu at (105.2, 70.2)
- added REF**: SMD Proto pad, Connectors:SMD_Proto_pad, F.Cu at (104.0, 70.2)
- added REF**: SMD Proto pad, Connectors:SMD_Proto_pad, F.Cu at (102.7, 70.2)
- added REF**: SMD Proto pad, Connectors:SMD_Proto_pad, F.Cu at (101.4, 70.2)
- added REF**: SMD Proto pad, Connectors:SMD_Proto_pad, F.Cu at (100.2, 70.2)
- added REF**: SMD Proto pad, Connectors:SMD_Proto_pad, F.Cu at (98.9, 70.2)
- added REF**: SMD Proto pad, Connectors:SMD_Proto_pad, F.Cu at (97.6, 70.2)
- added REF**: SMD Proto pad, Connectors:SMD_Proto_pad, F.Cu at (96.4, 70.2)
- added REF**: SMD Proto pad, Connectors:SMD_Proto_pad, F.Cu at (95.1, 70.2)
- added REF**: SMD Proto pad, Connectors:SMD_Proto_pad, B.Cu at (100.8, 74.6)
- added REF**: SMD Proto pad, Connectors:SMD_Proto_pad, F.Cu at (93.8, 70.2)
- added REF**: SMD Proto pad, Connectors:SMD_Proto_pad, F.Cu at (92.5, 70.2)
- added REF**: SMD Proto pad, Connectors:SMD_Proto_pad, F.Cu at (91.3, 70.2)
- added REF**: SMD Proto pad, Connectors:SMD_Proto_pad, F.Cu at (90.0, 70.2)
- added REF**: SMD Proto pad, Connectors:SMD_Proto_pad, F.Cu at (88.7, 70.2)
- added REF**: SMD Proto pad, Connectors:SMD_Proto_pad, F.Cu at (87.5, 70.2)
- added REF**: SMD Proto pad, Connectors:SMD_Proto_pad, F.Cu at (86.2, 70.2)
- added REF**: SMD Proto pad, Connectors:SMD_Proto_pad, F.Cu at (84.9, 70.2)
- added REF**: SMD Proto pad, Connectors:SMD_Proto_pad, F.Cu at (83.7, 70.2)
- added REF**: SMD Proto pad, Connectors:SMD_Proto_pad, F.Cu at (82.4, 70.2)
- added REF**: SMD Proto pad, Connectors:SMD_Proto_pad, B.Cu at (100.8, 73.4)
- added REF**: SMD Proto pad, Connectors:SMD_Proto_pad, F.Cu at (106.5, 67.7)
- added REF**: SMD Proto pad, Connectors:SMD_Proto_pad, F.Cu at (105.2, 67.7)
- added REF**: SMD Proto pad, Connectors:SMD_Proto_pad, F.Cu at (104.0, 67.7)
- added REF**: SMD Proto pad, Connectors:SMD_Proto_pad, F.Cu at (102.7, 67.7)
- added REF**: SMD Proto pad, Connectors:SMD_Proto_pad, F.Cu at (101.4, 67.7)
- added REF**: SMD Proto pad, Connectors:SMD_Proto_pad, F.Cu at (100.2, 67.7)
- added REF**: SMD Proto pad, Connectors:SMD_Proto_pad, F.Cu at (98.9, 67.7)
- added REF**: SMD Proto pad, Connectors:SMD_Proto_pad, F.Cu at (97.6, 67.7)
- added REF**: SMD Proto pad, Connectors:SMD_Proto_pad, F.Cu at (96.4, 67.7)
- added REF**: SMD Proto pad, Connectors:SMD_Proto_pad, F.Cu at (95.1, 67.7)
- added REF**: SMD Proto pad, Connectors:SMD_Proto_pad, B.Cu at (100.8, 72.1)
- added REF**: SMD Proto pad, Connectors:SMD_Proto_pad, F.Cu at (93.8, 67.7)
- added REF**: SMD Proto pad, Connectors:SMD_Proto_pad, F.Cu at (92.5, 67.7)
- added REF**: SMD Proto pad, Connectors:SMD_Proto_pad, F.Cu at (91.3, 67.7)
- added REF**: SMD Proto pad, Connectors:SMD_Proto_pad, F.Cu at (90.0, 67.7)
- added REF**: SMD Proto pad, Connectors:SMD_Proto_pad, F.Cu at (88.7, 67.7)
- added REF**: SMD Proto pad, Connectors:SMD_Proto_pad, F.Cu at (87.5, 67.7)
- added REF**: SMD Proto pad, Connectors:SMD_Proto_pad, F.Cu at (86.2, 67.7)
- added REF**: SMD Proto pad, Connectors:SMD_Proto_pad, F.Cu at (84.9, 67.7)
- added REF**: SMD Proto pad, Connectors:SMD_Proto_pad, F.Cu at (83.7, 67.7)
- added REF**: SMD Proto pad, Connectors:SMD_Proto_pad, F.Cu at (82.4, 67.7)
- added REF**: SMD Proto pad, Connectors:SMD_Proto_pad, B.Cu at (95.7, 82.3)
- added REF**: SMD Proto pad, Connectors:SMD_Proto_pad, B.Cu at (100.8, 70.8)
- added REF**: SMD Proto pad, Connectors:SMD_Proto_pad, F.Cu at (106.5, 65.1)
- added REF**: SMD Proto pad, Connectors:SMD_Proto_pad, F.Cu at (105.2, 65.1)
- added REF**: SMD Proto pad, Connectors:SMD_Proto_pad, F.Cu at (104.0, 65.1)
- added REF**: SMD Proto pad, Connectors:SMD_Proto_pad, F.Cu at (102.7, 65.1)
- added REF**: SMD Proto pad, Connectors:SMD_Proto_pad, F.Cu at (101.4, 65.1)
- added REF**: SMD Proto pad, Connectors:SMD_Proto_pad, F.Cu at (100.2, 65.1)
- added REF**: SMD Proto pad, Connectors:SMD_Proto_pad, F.Cu at (98.9, 65.1)
- added REF**: SMD Proto pad, Connectors:SMD_Proto_pad, F.Cu at (97.6, 65.1)
- added REF**: SMD Proto pad, Connectors:SMD_Proto_pad, F.Cu at (96.4, 65.1)
- added REF**: SMD Proto pad, Connectors:SMD_Proto_pad, F.Cu at (95.1, 65.1)
- added REF**: SMD Proto pad, Connectors:SMD_Proto_pad, B.Cu at (100.8, 69.6)
- added REF**: SMD Proto pad, Connectors:SMD_Proto_pad, F.Cu at (93.8, 65.1)
- added REF**: SMD Proto pad, Connectors:SMD_Proto_pad, F.Cu at (92.5, 65.1)
- added REF**: SMD Proto pad, Connectors:SMD_Proto_pad, F.Cu at (91.3, 65.1)
- added REF**: SMD Proto pad, Connectors:SMD_Proto_pad, F.Cu at (90.0, 65.1)
- added REF**: SMD Proto pad, Connectors:SMD_Proto_pad, F.Cu at (88.7, 65.1)
- added REF**: SMD Proto pad, Connectors:SMD_Proto_pad, F.Cu at (87.5, 65.1)
- added REF**: SMD Proto pad, Connectors:SMD_Proto_pad, F.Cu at (86.2, 65.1)
- added REF**: SMD Proto pad, Connectors:SMD_Proto_pad, F.Cu at (84.9, 65.1)
- added REF**: SMD Proto pad, Connectors:SMD_Proto_pad, F.Cu at (83.7, 65.1)
- added REF**: SMD Proto pad, Connectors:SMD_Proto_pad, F.Cu at (82.4, 65.1)
- added REF**: SMD Proto pad, Connectors:SMD_Proto_pad, B.Cu at (100.8, 68.3)
- added REF**: SMD Proto pad, Connectors:SMD_Proto_pad, F.Cu at (106.5, 62.6)
- added REF**: SMD Proto pad, Connectors:SMD_Proto_pad, F.Cu at (105.2, 62.6)
- added REF**: SMD Proto pad, Connectors:SMD_Proto_pad, F.Cu at (104.0, 62.6)
- added REF**: SMD Proto pad, Connectors:SMD_Proto_pad, F.Cu at (102.7, 62.6)
- added REF**: SMD Proto pad, Connectors:SMD_Proto_pad, F.Cu at (101.4, 62.6)
- added REF**: SMD Proto pad, Connectors:SMD_Proto_pad, F.Cu at (100.2, 62.6)
- added REF**: SMD Proto pad, Connectors:SMD_Proto_pad, F.Cu at (98.9, 62.6)
- added REF**: SMD Proto pad, Connectors:SMD_Proto_pad, F.Cu at (97.6, 62.6)
- added REF**: SMD Proto pad, Connectors:SMD_Proto_pad, F.Cu at (96.4, 62.6)
- added REF**: SMD Proto pad, Connectors:SMD_Proto_pad, F.Cu at (95.1, 62.6)
- added REF**: SMD Proto pad, Connectors:SMD_Proto_pad, B.Cu at (100.8, 67.0)
- added REF**: SMD Proto pad, Connectors:SMD_Proto_pad, F.Cu at (93.8, 62.6)
- added REF**: SMD Proto pad, Connectors:SMD_Proto_pad, F.Cu at (92.5, 62.6)
- added REF**: SMD Proto pad, Connectors:SMD_Proto_pad, F.Cu at (91.3, 62.6)
- added REF**: SMD Proto pad, Connectors:SMD_Proto_pad, F.Cu at (90.0, 62.6)
- added REF**: SMD Proto pad, Connectors:SMD_Proto_pad, F.Cu at (88.7, 62.6)
- added REF**: SMD Proto pad, Connectors:SMD_Proto_pad, F.Cu at (87.5, 62.6)
- added REF**: SMD Proto pad, Connectors:SMD_Proto_pad, F.Cu at (86.2, 62.6)
- added REF**: SMD Proto pad, Connectors:SMD_Proto_pad, F.Cu at (84.9, 62.6)
- added REF**: SMD Proto pad, Connectors:SMD_Proto_pad, F.Cu at (83.7, 62.6)
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Routing:
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- added copper zone on B.Cu, net GND
- added copper zone on F.Cu, net GND
Other:
- board outline added: 98 x 48 mm
- net class Default: via_dia 0.8 -> 0.5; via_drill 0.4 -> 0.3
- board text added: "0"
- board text added: "1"
- board text added: "2"
- board text added: "3"
- board text added: "4"
- board text added: "5"
- board text added: "6"
- board text added: "7"
- board text added: "8"
- board text added: "9"
- board text added: "A"
- board text added: "B"
- board text added: "C"
- board text added: "CLK"
- board text added: "D"
- board text added: "Designed by: Thomas Flummer"
- board text added: "Dev Edition"
- board text added: "E"
- board text added: "F"
- board text added: "G"
- board text added: "GND"
- board text added: "Geckonator"
- board text added: "H"
- board text added: "I"
- board text added: "IO"
- board text added: "J"
- board text added: "K"
- board text added: "L"
- board text added: "RX"
- board text added: "SCL"
- board text added: "SDA"
- board text added: "TX"
- board text added: "VCC"
- board text added: "X"
- board text added: "Y"
- board text added: "https://geckonator.dk"
