File: Geckonator Dev Edition.sch (KiCad schematic (older format))
At the start: 36 parts, among them J1 DEBUG, J2 LE UART, J3 I2C, J4 CONN_02X04, J5 CONN_02X04, J6 CONN_02X04, P1 USB_OTG, Q1 FDC6420C, SW1 BOOT, SW2 POWER, U1 EFM32HG322

Commit message: Added silkscreen, etc.
This corresponds to the first version produced

Signed-off-by: Thomas Flummer <tf@flummer.net>
Parts:
- removed BT?: Battery_Cell, symbol device:Battery_Cell
- removed C1, C2, C? (x3): 1uF, Capacitors_SMD:C_0805, symbol device:C
- removed C6: 4.7uF, Capacitors_SMD:C_0805, symbol device:C
- removed C? (x2): 100nF, symbol device:C
- removed C?: 10uF, symbol device:CP
- removed D1: LED_RGBA, Opto:RGBA_LED_SMD_0606, symbol Geckonator-Dev-Edition-rescue:LED_RGBA-RESCUE-Geckonator_Dev_Edition
- removed IC?: MAX1555, symbol maxim-ic:MAX1555
- removed P1: USB_OTG, Connectors:USB_Micro-B_10103594-0001LF, symbol Geckonator-Dev-Edition-rescue:USB_OTG-RESCUE-Bornhack_Make_Tradition_Badge-RESC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
- removed Q1: FDC6420C, TO_SOT_Packages_SMD:SuperSOT-6, symbol Semiconductors:FDC6420C
- removed Q?: FDC6331L, symbol Semiconductors:FDC6331L
- removed R1: 1.5K, Resistors_SMD:R_0805, symbol device:R
- removed R2: 1.2K, Resistors_SMD:R_0805, symbol device:R
- removed R3: 820, Resistors_SMD:R_0805, symbol device:R
- removed R4, R7: 4.7K, Resistors_SMD:R_0805, symbol device:R
- removed R5, R6: 15, Resistors_SMD:R_0805, symbol device:R
- removed R8: 6.8K, Resistors_SMD:R_0805, symbol device:R
- removed R?: 1M, Resistors_SMD:R_0805, symbol device:R
- removed SW1: BOOT, Buttons_Switches_SMD:SW_SPST_PTS645, symbol Geckonator-Dev-Edition-rescue:SW_PUSH-RESCUE-Geckonator_Dev_Edition
- removed SW2: POWER, Buttons_Switches_SMD:SW_SPST_PTS645, symbol Geckonator-Dev-Edition-rescue:SW_PUSH-RESCUE-Geckonator_Dev_Edition
- removed U?: MCP112T, symbol Semiconductors:MCP112T
- removed U?: NCP1117-3.3_TO252, TO_SOT_Packages_SMD:TO-252-2, symbol regul:NCP1117-3.3_TO252
- removed U?: USB_TYPE_C, symbol usb-type-c:USB_TYPE_C
- added C1, C2: CERAMIC-100NF-50V-10%-X7R_0603_, SeeedOPL-Capacitor-2016:C0603, symbol SeeedOPL-Capacitor-2016:CERAMIC-100NF-50V-10%-X7R_0603_
- added C3: CERAMIC-4.7UF-10V-10%-X5R_0603_, SeeedOPL-Capacitor-2016:C0603, symbol SeeedOPL-Capacitor-2016:CERAMIC-4.7UF-10V-10%-X5R_0603_
- added D1: LED-SMD-RED-DIFFUSED_0603_, SeeedOPL-LED-2016:LED-0603, symbol SeeedOPL-LED-2016:LED-SMD-RED-DIFFUSED_0603_
- added D2: SMD-LED-CLEAR-GREEN_0603_, SeeedOPL-LED-2016:LED-0603, symbol SeeedOPL-LED-2016:SMD-LED-CLEAR-GREEN_0603_
- added D3: SMD-LED-CLEAR-BLUE_0603_, SeeedOPL-LED-2016:LED-0603, symbol SeeedOPL-LED-2016:SMD-LED-CLEAR-BLUE_0603_
- added J7: BTNS, Pin_Headers:Pin_Header_Straight_1x04_Pitch2.54mm, symbol Geckonator-Dev-Edition-rescue:CONN_01X04-RESCUE-Geckonator_Dev_Edition
- added K1: BOOT, SeeedOPL-Switch-2016:SW4-SMD-6.0X6.0X5.0MM, symbol SeeedOPL-Switch-2016:SMD-SWITCH-TACTILE-SPST-NO_4P-D6.0MM_
- added K2: POWER, SeeedOPL-Switch-2016:SW4-SMD-6.0X6.0X5.0MM, symbol SeeedOPL-Switch-2016:SMD-SWITCH-TACTILE-SPST-NO_4P-D6.0MM_
- added R1: SMD-RES-1.5K-5%-1_10W_0603_, SeeedOPL-Resistor-2016:R0603, symbol SeeedOPL-Resistor-2016:SMD-RES-1.5K-5%-1_10W_0603_
- added R2, R3: SMD-RES-1K-5%-1_10W_0603_, SeeedOPL-Resistor-2016:R0603, symbol SeeedOPL-Resistor-2016:SMD-RES-1K-5%-1_10W_0603_
- added R4: SMD-RES-4.7K-5%-1_10W_0603_, SeeedOPL-Resistor-2016:R0603, symbol SeeedOPL-Resistor-2016:SMD-RES-4.7K-5%-1_10W_0603_
- added R5, R6: SMD-RES-22R-5%-1_10W_0603_, SeeedOPL-Resistor-2016:R0603, symbol SeeedOPL-Resistor-2016:SMD-RES-22R-5%-1_10W_0603_
- added USB1: MICRO-USB-SMD_ZX62-B-5PA_, SeeedOPL-Connector-2016:MICRO-USB5+6P-SMD-0.65-AB, symbol SeeedOPL-Connector-2016:MICRO-USB-SMD_ZX62-B-5PA_
Connections:
- net labels added: BUTTON_A, BUTTON_B, BUTTON_X, BUTTON_Y
- net labels removed: BATLOAD, DC_VIN, VBAT, VIN
- wire segments 178 -> 115
